File: micropad.kicad_pcb (KiCad board)
At the start: 2 copper layers, 79.4 x 66.1 mm, 19 parts

Commit message: Add files via upload
Parts:
- moved DEV1 2.58 mm to (111.5, 44.5)
Routing:
- net Net-(DEV1-D2): track 87.6 -> 90.5 mm
- net Net-(DEV1-D1): track 78.7 -> 81.4 mm
- net Net-(DEV1-D9): track 154.0 -> 156.6 mm
- net Net-(DEV1-D10): track 127.8 -> 130.4 mm
- net Net-(D3-K): track 143.4 -> 146.0 mm
- net Net-(D2-K): track 135.9 -> 138.5 mm
- net Net-(D1-K): track 97.0 -> 99.5 mm
- net Net-(E1-COM): track 125.6 -> 123.6 mm
- net Net-(DEV1-GND-Pad5): track 91.5 -> 92.9 mm
